File: sfp_module.kicad_sch (KiCad schematic)
At the start: 14 parts

Commit message: Replaced Mouser with LCSC Components
Parts:
- removed C202, C204, C205: (no value), symbol Device:C
- removed R202, R203, R204, R205: (no value), symbol Device:R
- added C302, C305: 100nF, Capacitor_SMD:C_0805_2012Metric, symbol Device:C
- added C304: 10uF, Capacitor_SMD:C_0805_2012Metric, symbol Device:C
- added R302, R303, R304, R305: 10k, Resistor_SMD:R_0805_2012Metric, symbol Device:R
- C301: renamed from C201; value (none) -> 10uF; footprint (none) -> Capacitor_SMD:C_0805_2012Metric; LCSC Part Number (none) -> C386084; Mouser Link https://www.mouser.de/ProductDetail/Samsung-Electro-Mechani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 -> (none); Mouser Part Number 187-CL21A106KQFNNNG -> (none); Part Number CL21A106KQFNNNG -> (none)
- C303: renamed from C203; value (none) -> 100nF; footprint (none) -> Capacitor_SMD:C_0805_2012Metric; LCSC Part Number (none) -> C396718; Mouser Link https://www.mouser.de/ProductDetail/AVX/06033C104KAT4A?qs=8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 -> (none); Mouser Part Number 581-06033C104KAT4A -> (none); Part Number 06033C104KAT4A -> (none)
- J301: renamed from J201; value (none) -> SFP; footprint (none) -> Connector:Connector_SFP_and_Cage; LCSC Part Number (none) -> C277615; Mouser Link https://www.mouser.de/ProductDetail/Molex/74441-0001?qs=%2F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 -> (none); Mouser Part Number 538-74441-0001 -> (none); Part Number 74441-0001 -> (none)
- L301: renamed from L201; value (none) -> 1uH; footprint (none) -> Inductor_SMD:L_0805_2012Metric; LCSC Part Number (none) -> C162587; Mouser Link https://www.mouser.de/ProductDetail/Taiyo-Yuden/MCKK2012T1R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 -> (none); Mouser Part Number 963-MCKK2012T1R0M -> (none); Part Number MCKK2012T1R0M -> (none)
- L302: renamed from L202; value (none) -> 1uH; footprint (none) -> Inductor_SMD:L_0805_2012Metric; LCSC Part Number (none) -> C162587; Mouser Link https://www.mouser.de/ProductDetail/Taiyo-Yuden/MCKK2012T1R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 -> (none); Mouser Part Number 963-MCKK2012T1R0M -> (none); Part Number MCKK2012T1R0M -> (none)
- N2: renamed from N?; value (none) -> Housing_Pad; LCSC Part Number (none) -> C2897292
- R301: renamed from R201; value (none) -> 10k; footprint (none) -> Resistor_SMD:R_0805_2012Metric; LCSC Part Number (none) -> C17414; Mouser Link https://www.mouser.de/ProductDetail/Welwyn-Components-TT-El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 -> (none); Mouser Part Number 756-WCR0603-10KFA -> (none); Part Number WCR0603-10KFA -> (none)
Connections:
- net 3.3V: now also C302.1
- net GND: now also C302.2, C304.2, C305.2
- net RX_LOS: now also R304.1
- net TX_FAULT: now also R305.2
- net VCC_R: now also C304.1, C305.1
- net VCC_T: now also R302.2, R303.2, R304.2, R305.1
- net at J301.4 (MOD_DEF2): now also R303.1
- net at J301.5 (MOD_DEF1): now also R302.1
Other:
- moved on the sheet: C301, R301

Commit message: Added I2C pins
Parts:
- R301, R302, R303, R304, R305: value 10k -> (none); footprint Resistor_SMD:R_0805_2012Metric -> (none); LCSC Part Number C17414 -> C17673
Connections:
- net at R303.1: now also J301.6 (MOD_DEF0); no longer J301.4 (MOD_DEF2)
- net MOD_DEF1_SCL: now reaches J301.5 (MOD_DEF1), R302.1
- net MOD_DEF2_SDA: now reaches R301.1
- net MOD_DEF2_SDA: now also J301.4 (MOD_DEF2); no longer J301.6 (MOD_DEF0)
Other:
- moved on the sheet: N2

Commit message: WIP
Parts:
- C303: value 100nF -> (none); footprint Capacitor_SMD:C_0805_2012Metric -> (none)
- L301, L302: value 1uH -> (none); footprint Inductor_SMD:L_0805_2012Metric -> (none)
- R302, R303, R304, R305: value (none) -> 4.7k; footprint (none) -> Resistor_SMD:R_0805_2012Metric
Changed lines of the file:
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@@
     (in_bom yes) (on_board yes)
     (property "Reference" "L301" (id 0) (at 96.52 67.564 90))
-    (property "Value" "1uH" (id 1) (at 96.52 69.8754 90))
-    (property "Footprint" "Inductor_SMD:L_0805_2012Metric" (id 2) (at 96.52 72.39 0)
+    (property "Value" "" (id 1) (at 96.52 69.8754 90))
+    (property "Footprint" "" (id 2) (at 96.52 72.39 0)
       (effects (font (size 1.27 1.27)) hide)
     )
@@
     (in_bom yes) (on_board yes)
     (property "Reference" "L302" (id 0) (at 96.52 86.614 90))
-    (property "Value" "1uH" (id 1) (at 96.52 88.9254 90))
-    (property "Footprint" "Inductor_SMD:L_0805_2012Metric" (id 2) (at 96.52 91.44 0)
+    (property "Value" "" (id 1) (at 96.52 88.9254 90))
+    (property "Footprint" "" (id 2) (at 96.52 91.44 0)
       (effects (font (size 1.27 1.27)) hide)
     )
@@
       (effects (font (size 1.27 1.27)) (justify left))
     )
-    (property "Value" "100nF" (id 1) (at 108.331 79.883 0)
-      (effects (font (size 1.27 1.27)) (justify left))
-    )
-    (property "Footprint" "Capacitor_SMD:C_0805_2012Metric" (id 2) (at 106.3752 82.55 0)
+    (property "Value" "" (id 1) (at 108.331 79.883 0)
+      (effects (font (size 1.27 1.27)) (justify left))
+    )
+    (property "Footprint" "" (id 2) (at 106.3752 82.55 0)
       (effects (font (size 1.27 1.27)) hide)
     )
@@
       (effects (font (size 1.27 1.27)) (justify left))
     )
-    (property "Value" "" (id 1) (at 213.868 68.707 0)
-      (effects (font (size 1.27 1.27)) (justify left))
-    )
-    (property "Footprint" "" (id 2) (at 210.312 69.85 90)
+    (property "Value" "4.7k" (id 1) (at 213.868 68.707 0)
+      (effects (font (size 1.27 1.27)) (justify left))
+    )
+    (property "Footprint" "Resistor_SMD:R_0805_2012Metric" (id 2) (at 210.312 69.85 90)
       (effects (font (size 1.27 1.27)) hide)
     )
@@
       (effects (font (size 1.27 1.27)) (justify left))
     )
-    (property "Value" "" (id 1) (at 178.308 68.707 0)
-      (effects (font (size 1.27 1.27)) (justify left))
-    )
-    (property "Footprint" "" (id 2) (at 174.752 69.85 90)
+    (property "Value" "4.7k" (id 1) (at 178.308 68.707 0)
+      (effects (font (size 1.27 1.27)) (justify left))
+    )
+    (property "Footprint" "Resistor_SMD:R_0805_2012Metric" (id 2) (at 174.752 69.85 90)
       (effects (font (size 1.27 1.27)) hide)
     )
@@
       (effects (font (size 1.27 1.27)) (justify left))
     )
-    (property "Value" "" (id 1) (at 213.868 104.267 0)
-      (effects (font (size 1.27 1.27)) (justify left))
-    )
-    (property "Footprint" "" (id 2) (at 210.312 105.41 90)
+    (property "Value" "4.7k" (id 1) (at 213.868 104.267 0)
+      (effects (font (size 1.27 1.27)) (justify left))
+    )
+    (property "Footprint" "Resistor_SMD:R_0805_2012Metric" (id 2) (at 210.312 105.41 90)
       (effects (font (size 1.27 1.27)) hide)
     )
@@
       (effects (font (size 1.27 1.27)) (justify left))
     )
-    (property "Value" "" (id 1) (at 169.418 68.707 0)
-      (effects (font (size 1.27 1.27)) (justify left))
-    )
-    (property "Footprint" "" (id 2) (at 165.862 69.85 90)
-      (effects (font (size 1.27 1.27)) hide)
-    )
+    (property "Value" "4.7k" (id 1) (at 169.418 68.707 0)
+      (effects (font (size 1.27 1.27)) (justify left))
+    )
+    (property "Footprint" "Resistor_SMD:R_0805_2012Metric" (id 2) (at 165.862 69.85 90)
+      (effects (font (size 1.27 1.27)) hide)
+    )

Commit message: Finished PCB and renamed it
Parts:
- C303: value (none) -> 100nF; footprint (none) -> Capacitor_SMD:C_0805_2012Metric
- L301, L302: value (none) -> 1uH; footprint (none) -> Inductor_SMD:L_1008_2520Metric
- N2: footprint (none) -> TestPoint:TestPoint_Pad_D1.0mm; Mouser Link https://www.mouser.de/ProductDetail/Molex/74737-0010?qs=%2F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 -> (none); Mouser Part Number 538-74737-0010 -> (none); Part Number 74737-0010 -> (none)
- R301: value (none) -> 4.7k; footprint (none) -> Resistor_SMD:R_0805_2012Metric
- R302, R303, R304: LCSC Part Number C17673 -> C17673
Changed lines of the file:
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@@
       (effects (font (size 1.27 1.27)) hide)
     )
-    (property "Datasheet" "" (id 3) (at 184.15 71.12 0)
+    (property "Datasheet" "~" (id 3) (at 184.15 71.12 0)
       (effects (font (size 1.27 1.27)) hide)
     )
@@
       (effects (font (size 1.27 1.27)) (justify left))
     )
-    (property "Value" "" (id 1) (at 160.528 68.707 0)
-      (effects (font (size 1.27 1.27)) (justify left))
-    )
-    (property "Footprint" "" (id 2) (at 156.972 69.85 90)
+    (property "Value" "4.7k" (id 1) (at 160.528 68.707 0)
+      (effects (font (size 1.27 1.27)) (justify left))
+    )
+    (property "Footprint" "Resistor_SMD:R_0805_2012Metric" (id 2) (at 156.972 69.85 90)
       (effects (font (size 1.27 1.27)) hide)
     )
@@
     (in_bom yes) (on_board yes)
     (property "Reference" "L301" (id 0) (at 96.52 67.564 90))
-    (property "Value" "" (id 1) (at 96.52 69.8754 90))
-    (property "Footprint" "" (id 2) (at 96.52 72.39 0)
-      (effects (font (size 1.27 1.27)) hide)
-    )
-    (property "Datasheet" "" (id 3) (at 96.52 72.39 0)
+    (property "Value" "1uH" (id 1) (at 96.52 69.8754 90))
+    (property "Footprint" "Inductor_SMD:L_1008_2520Metric" (id 2) (at 96.52 72.39 0)
+      (effects (font (size 1.27 1.27)) hide)
+    )
+    (property "Datasheet" "~" (id 3) (at 96.52 72.39 0)
       (effects (font (size 1.27 1.27)) hide)
     )
@@
     (in_bom yes) (on_board yes)
     (property "Reference" "L302" (id 0) (at 96.52 86.614 90))
-    (property "Value" "" (id 1) (at 96.52 88.9254 90))
-    (property "Footprint" "" (id 2) (at 96.52 91.44 0)
-      (effects (font (size 1.27 1.27)) hide)
-    )
-    (property "Datasheet" "" (id 3) (at 96.52 91.44 0)
+    (property "Value" "1uH" (id 1) (at 96.52 88.9254 90))
+    (property "Footprint" "Inductor_SMD:L_1008_2520Metric" (id 2) (at 96.52 91.44 0)
+      (effects (font (size 1.27 1.27)) hide)
+    )
+    (property "Datasheet" "~" (id 3) (at 96.52 91.44 0)
       (effects (font (size 1.27 1.27)) hide)
     )
@@
       (effects (font (size 1.27 1.27)) (justify left))
     )
-    (property "Value" "" (id 1) (at 108.331 79.883 0)
-      (effects (font (size 1.27 1.27)) (justify left))
-    )
-    (property "Footprint" "" (id 2) (at 106.3752 82.55 0)
+    (property "Value" "100nF" (id 1) (at 108.331 79.883 0)
+      (effects (font (size 1.27 1.27)) (justify left))
+    )
+    (property "Footprint" "Capacitor_SMD:C_0805_2012Metric" (id 2) (at 106.3752 82.55 0)
       (effects (font (size 1.27 1.27)) hide)
     )
@@
       (effects (font (size 1.27 1.27)) (justify left))
     )
-    (property "Footprint" "" (id 2) (at 193.675 44.45 0)
-      (effects (font (size 1.27 1.27)) hide)
-    )
-    (property "Datasheet" "https://www.mouser.de/datasheet/2/276/1/0747370010_EMI_CAGES-1373392.pdf" (id 3) (at 193.675 44.45 0)
-      (effects (font (size 1.27 1.27)) hide)
-    )
-    (property "Mouser Link" "https://www.mouser.de/ProductDetail/Molex/74737-0010?qs=%2Fha2pyFadujrqsB3QNYa%252BMTp8Wab2kbqfDhy%2FouEo9Y%3D" (id 4) (at 191.77 45.72 0)
-      (effects (font (size 1.27 1.27)) hide)
-    )
-    (property "Mouser Part Number" "538-74737-0010" (id 5) (at 191.77 45.72 0)
-      (effects (font (size 1.27 1.27)) hide)
-    )
-    (property "Part Number" "74737-0010" (id 6) (at 191.77 45.72 0)
+    (property "Footprint" "TestPoint:TestPoint_Pad_D1.0mm" (id 2) (at 193.675 44.45 0)
+      (effects (font (size 1.27 1.27)) hide)
+    )
+    (property "Datasheet" "~" (id 3) (at 193.675 44.45 0)
       (effects (font (size 1.27 1.27)) hide)
     )
@@
       (effects (font (size 1.27 1.27)) hide)
     )
-    (property "LCSC Part Number" " C17673" (id 5) (at 212.09 69.85 0)
+    (property "LCSC Part Number" "C17673" (id 5) (at 212.09 69.85 0)
       (effects (font (size 1.27 1.27)) hide)
     )
@@
       (effects (font (size 1.27 1.27)) hide)
     )
-    (property "LCSC Part Number" " C17673" (id 5) (at 176.53 69.85 0)
+    (property "LCSC Part Number" "C17673" (id 5) (at 176.53 69.85 0)
       (effects (font (size 1.27 1.27)) hide)
     )
@@
       (effects (font (size 1.27 1.27)) hide)
     )
-    (property "LCSC Part Number" " C17673" (id 5) (at 167.64 69.85 0)
-      (effects (font (size 1.27 1.27)) hide)
-    )
+    (property "LCSC Part Number" "C17673" (id 5) (at 167.64 69.85 0)
+      (effects (font (size 1.27 1.27)) hide)
+    )
